File: OpenHealth_Hardware/OpenHealth_rj45v2.brd (EAGLE design)
At the start: 128.2 x 44.1 mm, 7 parts

Commit message: se añadio el git ignore se trabajo en un escudo version oshpark y se sigue trabajando en la tarjeta principal
Parts:
- added U$1: (no value), SparkFun-Aesthetics:OSHW-LOGO-S_COPPER
- moved CONECTOR_A 2.54 mm to (115.6, 24.1)
- moved CONECTOR_B 2.54 mm to (11.4, 24.1)
Routing:
- net GND: track 343.8 -> 231.7 mm
- net 3.3V: track 138.6 -> 90.7 mm, vias 5 -> 0
- net BPM_RX: track 133.0 -> 97.9 mm
- net D12: track 68.6 -> 39.8 mm
- net BPM_TX: track 114.5 -> 88.4 mm
- net SALIDA_D6: track 98.6 -> 74.8 mm
- net D11: track 58.1 -> 35.5 mm
- net LCA_YLW: track 50.6 -> 30.1 mm
- net A0: track 73.2 -> 53.1 mm
- net RA: track 38.9 -> 19.6 mm
- net LCA_GRN: track 40.5 -> 24.0 mm
- net LCA_WHT: track 24.9 -> 17.8 mm
- net LA: track 17.8 -> 13.4 mm
- net LCA_BLK: track 16.2 -> 11.8 mm
- net VIN: track 96.9 -> 100.9 mm, vias 5 -> 0
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Other:
- board size 128.2 x 44.1 mm -> 119.4 x 20 mm
- board text added: "ALSW Project Open Health V2"
